Commit message: refine gr1t2 mjcf model

File: models/GR1/GR1T1/urdf/GR1T1_raw.urdf (robot description, URDF)
Before this commit: robot GR1T1, 33 links, 32 joints
Joints:
- joint l_hip_roll: limit lower=-0.09 upper=0.79 effort=100 velocity=12.15 -> lower=-0.09 upper=0.79 effort=80 velocity=12.15
- joint l_hip_yaw: limit lower=-0.7 upper=0.7 effort=82.5 velocity=16.76 -> lower=-0.7 upper=0.7 effort=60 velocity=16.76
- joint r_hip_roll: limit lower=-0.79 upper=0.09 effort=100 velocity=12.15 -> lower=-0.79 upper=0.09 effort=80 velocity=12.15
- joint r_hip_yaw: limit lower=-0.7 upper=0.7 effort=82.5 velocity=16.76 -> lower=-0.7 upper=0.7 effort=60 velocity=16.76
- joint waist_pitch: limit lower=-0.52 upper=1.22 effort=82.5 velocity=16.76 -> lower=-0.52 upper=1.22 effort=60 velocity=16.76
- joint waist_roll: limit lower=-0.7 upper=0.7 effort=82.5 velocity=16.76 -> lower=-0.7 upper=0.7 effort=60 velocity=16.76
- joint waist_yaw: limit lower=-1.05 upper=1.05 effort=82.5 velocity=16.76 -> lower=-1.05 upper=1.05 effort=60 velocity=16.76

File: models/GR1/GR1T2/urdf/GR1T2_raw.urdf (robot description, URDF)
Before this commit: robot GR1T2, 35 links, 34 joints
Links:
- link l_foot_pitch: geometry collision mesh filename=../meshes/l_foot_pitch.STL; visual mesh filename=../meshes/l_foot_pitch.STL
- link l_foot_roll: geometry collision mesh filename=../meshes/l_foot_roll.STL; visual mesh filename=../meshes/l_foot_roll.STL
- link l_hand_pitch: geometry collision mesh filename=../meshes/l_hand_pitch.STL; visual mesh filename=../meshes/l_hand_pitch.STL
- link l_hand_roll: geometry collision mesh filename=../meshes/l_hand_roll.STL; visual mesh filename=../meshes/l_hand_roll.STL
- link l_hand_yaw: geometry collision mesh filename=../meshes/l_hand_yaw.STL; visual mesh filename=../meshes/l_hand_yaw.STL
- link l_lower_arm_pitch: geometry collision mesh filename=../meshes/l_lower_arm_pitch.STL; visual mesh filename=../meshes/l_lower_arm_pitch.STL
- link l_shank_pitch: geometry collision mesh filename=../meshes/l_shank_pitch.STL; visual mesh filename=../meshes/l_shank_pitch.STL
- link l_thigh_pitch: geometry collision mesh filename=../meshes/l_thigh_pitch.STL; visual mesh filename=../meshes/l_thigh_pitch.STL
- link l_thigh_roll: geometry collision mesh filename=../meshes/l_thigh_roll.STL; visual mesh filename=../meshes/l_thigh_roll.STL
- link l_thigh_yaw: geometry collision mesh filename=../meshes/l_thigh_yaw.STL; visual mesh filename=../meshes/l_thigh_yaw.STL
- link l_upper_arm_pitch: geometry collision mesh filename=../meshes/l_upper_arm_pitch.STL; visual mesh filename=../meshes/l_upper_arm_pitch.STL
- link l_upper_arm_roll: geometry collision mesh filename=../meshes/l_upper_arm_roll.STL; visual mesh filename=../meshes/l_upper_arm_roll.STL
- link l_upper_arm_yaw: geometry collision mesh filename=../meshes/l_upper_arm_yaw.STL; visual mesh filename=../meshes/l_upper_arm_yaw.STL
- link link_head_pitch: geometry collision mesh filename=../meshes/head_yaw.STL; visual mesh filename=../meshes/head_yaw.STL
- link link_head_roll: geometry collision mesh filename=../meshes/head_roll.STL; visual mesh filename=../meshes/head_roll.STL
- link link_head_yaw: geometry collision mesh filename=../meshes/head_pitch.STL; visual mesh filename=../meshes/head_pitch.STL
- link link_waist_pitch: geometry collision mesh filename=../meshes/waist_roll.STL; visual mesh filename=../meshes/waist_roll.STL
- link link_waist_roll: geometry collision mesh filename=../meshes/waist_roll.STL; visual mesh filename=../meshes/waist_roll.STL
- link link_waist_yaw: geometry collision mesh filename=../meshes/waist_yaw.STL; visual mesh filename=../meshes/waist_yaw.STL
- link r_foot_pitch: geometry collision mesh filename=../meshes/r_foot_pitch.STL; visual mesh filename=../meshes/r_foot_pitch.STL
- link r_foot_roll: geometry collision mesh filename=../meshes/r_foot_roll.STL; visual mesh filename=../meshes/r_foot_roll.STL
- link r_hand_pitch: geometry collision mesh filename=../meshes/r_hand_pitch.STL; visual mesh filename=../meshes/r_hand_pitch.STL
- link r_hand_roll: geometry collision mesh filename=../meshes/r_hand_roll.STL; visual mesh filename=../meshes/r_hand_roll.STL
- link r_hand_yaw: geometry collision mesh filename=../meshes/r_hand_yaw.STL; visual mesh filename=../meshes/r_hand_yaw.STL
- link r_lower_arm_pitch: geometry collision mesh filename=../meshes/r_lower_arm_pitch.STL; visual mesh filename=../meshes/r_lower_arm_pitch.STL
- link r_shank_pitch: geometry collision mesh filename=../meshes/r_shank_pitch.STL; visual mesh filename=../meshes/r_shank_pitch.STL
- link r_thigh_pitch: geometry collision mesh filename=../meshes/r_thigh_pitch.STL; visual mesh filename=../meshes/r_thigh_pitch.STL
- link r_thigh_roll: geometry collision mesh filename=../meshes/r_thigh_roll.STL; visual mesh filename=../meshes/r_thigh_roll.STL
- link r_thigh_yaw: geometry collision mesh filename=../meshes/r_thigh_yaw.STL; visual mesh filename=../meshes/r_thigh_yaw.STL
- link r_upper_arm_pitch: geometry collision mesh filename=../meshes/r_upper_arm_pitch.STL; visual mesh filename=../meshes/r_upper_arm_pitch.STL
- link r_upper_arm_roll: geometry collision mesh filename=../meshes/r_upper_arm_roll.STL; visual mesh filename=../meshes/r_upper_arm_roll.STL
- link r_upper_arm_yaw: geometry collision mesh filename=../meshes/r_upper_arm_yaw.STL; visual mesh filename=../meshes/r_upper_arm_yaw.STL
Joints:
- joint joint_head_pitch: origin xyz=0.000999999999997045 -0.000225512658326668 0.144786985472057 rpy=0 0 0 -> xyz=0.000999999999997045 -0.000160512658326668 0.144786985472057 rpy=0 0 0
- joint joint_waist_pitch: limit lower=-0.52 upper=1.22 effort=66 velocity=16.76 -> lower=-0.52 upper=1.22 effort=60 velocity=16.76
- joint joint_waist_roll: limit lower=-0.7 upper=0.7 effort=66 velocity=16.76 -> lower=-0.7 upper=0.7 effort=60 velocity=16.76
- joint joint_waist_yaw: limit lower=-1.05 upper=1.05 effort=66 velocity=16.76 -> lower=-1.05 upper=1.05 effort=60 velocity=16.76
- joint l_hip_pitch: limit lower=-1.75 upper=0.7 effort=225 velocity=37.38 -> lower=-1.75 upper=0.7 effort=160 velocity=37.38
- joint l_hip_roll: limit lower=-0.09 upper=0.79 effort=48 velocity=12.15 -> lower=-0.09 upper=0.79 effort=80 velocity=12.15
- joint l_hip_yaw: limit lower=-0.7 upper=0.7 effort=66 velocity=16.76 -> lower=-0.7 upper=0.7 effort=60 velocity=16.76
- joint l_knee_pitch: limit lower=-0.09 upper=1.92 effort=225 velocity=37.38 -> lower=-0.09 upper=1.92 effort=160 velocity=37.38
- joint r_hip_pitch: limit lower=-1.75 upper=0.7 effort=225 velocity=37.38 -> lower=-1.75 upper=0.7 effort=160 velocity=37.38
- joint r_hip_roll: limit lower=-0.79 upper=0.09 effort=48 velocity=12.15 -> lower=-0.79 upper=0.09 effort=80 velocity=12.15
- joint r_hip_yaw: limit lower=-0.7 upper=0.7 effort=66 velocity=16.76 -> lower=-0.7 upper=0.7 effort=60 velocity=16.76
- joint r_knee_pitch: limit lower=-0.09 upper=1.92 effort=225 velocity=37.38 -> lower=-0.09 upper=1.92 effort=160 velocity=37.38
