Commit message: update README.md

File: models/GR1/GR1T2/urdf/GR1T2_raw.urdf (robot description, URDF)
Before this commit: robot GR1T2, 35 links, 34 joints
Links:
- link base: geometry collision mesh filename=../meshes/base.STL; visual mesh filename=../meshes/base.STL
- link l_foot_pitch: geometry collision mesh filename=../meshes/Lleg5.STL; visual mesh filename=../meshes/Lleg5.STL
- link l_foot_roll: geometry collision mesh filename=../meshes/Lleg6.STL; visual mesh filename=../meshes/Lleg6.STL
- link l_hand_pitch: geometry collision mesh filename=../meshes/Larm7.STL; visual mesh filename=../meshes/Larm7.STL
- link l_hand_roll: geometry collision mesh filename=../meshes/Larm6.STL; visual mesh filename=../meshes/Larm6.STL
- link l_hand_yaw: geometry collision mesh filename=../meshes/Larm5.STL; visual mesh filename=../meshes/Larm5.STL
- link l_lower_arm_pitch: geometry collision mesh filename=../meshes/Larm4.STL; visual mesh filename=../meshes/Larm4.STL
- link l_shank_pitch: geometry collision mesh filename=../meshes/Lleg4.STL; visual mesh filename=../meshes/Lleg4.STL
- link l_thigh_pitch: geometry collision mesh filename=../meshes/Lleg3.STL; visual mesh filename=../meshes/Lleg3.STL
- link l_thigh_roll: geometry collision mesh filename=../meshes/Lleg1.STL; visual mesh filename=../meshes/Lleg1.STL
- link l_thigh_yaw: geometry collision mesh filename=../meshes/Lleg2.STL; visual mesh filename=../meshes/Lleg2.STL
- link l_upper_arm_pitch: geometry collision mesh filename=../meshes/Larm1.STL; visual mesh filename=../meshes/Larm1.STL
- link l_upper_arm_roll: geometry collision mesh filename=../meshes/Larm2.STL; visual mesh filename=../meshes/Larm2.STL
- link l_upper_arm_yaw: geometry collision mesh filename=../meshes/Larm3.STL; visual mesh filename=../meshes/Larm3.STL
- link link_head_pitch: geometry collision mesh filename=../meshes/head3.STL; visual mesh filename=../meshes/head3.STL
- link link_head_roll: geometry collision mesh filename=../meshes/head2.STL; visual mesh filename=../meshes/head2.STL
- link link_head_yaw: geometry collision mesh filename=../meshes/head1.STL; visual mesh filename=../meshes/head1.STL
- link link_waist_pitch: geometry collision mesh filename=../meshes/waist2.STL; visual mesh filename=../meshes/waist2.STL
- link link_waist_roll: geometry collision mesh filename=../meshes/waist1.STL; visual mesh filename=../meshes/waist1.STL
- link link_waist_yaw: geometry collision mesh filename=../meshes/waist3.STL; visual mesh filename=../meshes/waist3.STL
- link r_foot_pitch: geometry collision mesh filename=../meshes/Rleg5.STL; visual mesh filename=../meshes/Rleg5.STL
- link r_foot_roll: geometry collision mesh filename=../meshes/Rleg6.STL; visual mesh filename=../meshes/Rleg6.STL
- link r_hand_pitch: geometry collision mesh filename=../meshes/Rarm7.STL; visual mesh filename=../meshes/Rarm7.STL
- link r_hand_roll: geometry collision mesh filename=../meshes/Rarm6.STL; visual mesh filename=../meshes/Rarm6.STL
- link r_hand_yaw: geometry collision mesh filename=../meshes/Rarm5.STL; visual mesh filename=../meshes/Rarm5.STL
- link r_lower_arm_pitch: geometry collision mesh filename=../meshes/Rarm4.STL; visual mesh filename=../meshes/Rarm4.STL
- link r_shank_pitch: geometry collision mesh filename=../meshes/Rleg4.STL; visual mesh filename=../meshes/Rleg4.STL
- link r_thigh_pitch: geometry collision mesh filename=../meshes/Rleg3.STL; visual mesh filename=../meshes/Rleg3.STL
- link r_thigh_roll: geometry collision mesh filename=../meshes/Rleg1.STL; visual mesh filename=../meshes/Rleg1.STL
- link r_thigh_yaw: geometry collision mesh filename=../meshes/Rleg2.STL; visual mesh filename=../meshes/Rleg2.STL
- link r_upper_arm_pitch: geometry collision mesh filename=../meshes/Rarm1.STL; visual mesh filename=../meshes/Rarm1.STL
- link r_upper_arm_roll: geometry collision mesh filename=../meshes/Rarm2.STL; visual mesh filename=../meshes/Rarm2.STL
- link r_upper_arm_yaw: geometry collision mesh filename=../meshes/Rarm3.STL; visual mesh filename=../meshes/Rarm3.STL

Commit message: Update GR1T2_raw.urdf

File: models/GR1/GR1T2/urdf/GR1T2_raw.urdf (robot description, URDF)
Before this commit: robot GR1T2, 35 links, 34 joints
Links:
- removed link l_foot_pitch
- removed link l_foot_roll
- removed link l_hand_pitch
- removed link l_hand_roll
- removed link l_hand_yaw
- removed link l_lower_arm_pitch
- removed link l_thigh_pitch
- removed link l_thigh_yaw
- removed link l_upper_arm_pitch
- removed link l_upper_arm_roll
- removed link l_upper_arm_yaw
- removed link r_foot_pitch
- removed link r_foot_roll
- removed link r_hand_pitch
- removed link r_hand_roll
- removed link r_hand_yaw
- removed link r_lower_arm_pitch
- removed link r_shank_pitch
- removed link r_thigh_pitch
- removed link r_thigh_roll
- removed link r_thigh_yaw
- removed link r_upper_arm_pitch
- removed link r_upper_arm_roll
- removed link r_upper_arm_yaw
- added link link_left_foot_pitch, mass 0.049737; collision mesh filename=../meshes/l_foot_pitch.STL; visual mesh filename=../meshes/l_foot_pitch.STL
- added link link_left_foot_roll, mass 0.59122118; collision mesh filename=../meshes/l_foot_roll.STL; visual mesh filename=../meshes/l_foot_roll.STL
- added link link_left_hand_pitch, mass 0.54891; collision mesh filename=../meshes/l_hand_pitch.STL; visual mesh filename=../meshes/l_hand_pitch.STL
- added link link_left_hand_roll, mass 0.0054351; collision mesh filename=../meshes/l_hand_roll.STL; visual mesh filename=../meshes/l_hand_roll.STL
- added link link_left_hand_yaw, mass 1.2684; collision mesh filename=../meshes/l_hand_yaw.STL; visual mesh filename=../meshes/l_hand_yaw.STL
- added link link_left_lower_arm_pitch, mass 0.059535; collision mesh filename=../meshes/l_lower_arm_pitch.STL; visual mesh filename=../meshes/l_lower_arm_pitch.STL
- added link link_left_thigh_pitch, mass 6.1575; collision mesh filename=../meshes/l_thigh_pitch.STL; visual mesh filename=../meshes/l_thigh_pitch.STL
- added link link_left_thigh_yaw, mass 3.9947; collision mesh filename=../meshes/l_thigh_yaw.STL; visual mesh filename=../meshes/l_thigh_yaw.STL
- added link link_left_upper_arm_pitch, mass 0.78809; collision mesh filename=../meshes/l_upper_arm_pitch.STL; visual mesh filename=../meshes/l_upper_arm_pitch.STL
- added link link_left_upper_arm_roll, mass 0.1786; collision mesh filename=../meshes/l_upper_arm_roll.STL; visual mesh filename=../meshes/l_upper_arm_roll.STL
- added link link_left_upper_arm_yaw, mass 0.98085; collision mesh filename=../meshes/l_upper_arm_yaw.STL; visual mesh filename=../meshes/l_upper_arm_yaw.STL
- added link link_right_foot_pitch, mass 0.049737; collision mesh filename=../meshes/r_foot_pitch.STL; visual mesh filename=../meshes/r_foot_pitch.STL
- added link link_right_foot_roll, mass 0.59122; collision mesh filename=../meshes/r_foot_roll.STL; visual mesh filename=../meshes/r_foot_roll.STL
- added link link_right_hand_pitch, mass 0.54891; collision mesh filename=../meshes/r_hand_pitch.STL; visual mesh filename=../meshes/r_hand_pitch.STL
- added link link_right_hand_roll, mass 0.0054351; collision mesh filename=../meshes/r_hand_roll.STL; visual mesh filename=../meshes/r_hand_roll.STL
- added link link_right_hand_yaw, mass 1.2684; collision mesh filename=../meshes/r_hand_yaw.STL; visual mesh filename=../meshes/r_hand_yaw.STL
- added link link_right_lower_arm_pitch, mass 0.059535; collision mesh filename=../meshes/r_lower_arm_pitch.STL; visual mesh filename=../meshes/r_lower_arm_pitch.STL
- added link link_right_shank_pitch, mass 2.4196; collision mesh filename=../meshes/r_shank_pitch.STL; visual mesh filename=../meshes/r_shank_pitch.STL
- added link link_right_thigh_pitch, mass 6.1575; collision mesh filename=../meshes/r_thigh_pitch.STL; visual mesh filename=../meshes/r_thigh_pitch.STL
- added link link_right_thigh_roll, mass 1.2408; collision mesh filename=../meshes/r_thigh_roll.STL; visual mesh filename=../meshes/r_thigh_roll.STL
- added link link_right_thigh_yaw, mass 3.9947; collision mesh filename=../meshes/r_thigh_yaw.STL; visual mesh filename=../meshes/r_thigh_yaw.STL
- added link link_right_upper_arm_pitch, mass 0.78809; collision mesh filename=../meshes/r_upper_arm_pitch.STL; visual mesh filename=../meshes/r_upper_arm_pitch.STL
- added link link_right_upper_arm_roll, mass 0.1786; collision mesh filename=../meshes/r_upper_arm_roll.STL; visual mesh filename=../meshes/r_upper_arm_roll.STL
- added link link_right_upper_arm_yaw, mass 0.98085; collision mesh filename=../meshes/r_upper_arm_yaw.STL; visual mesh filename=../meshes/r_upper_arm_yaw.STL
Joints:
- removed joint l_ankle_pitch
- removed joint l_ankle_roll
- removed joint l_elbow_pitch
- removed joint l_hip_pitch
- removed joint l_hip_roll
- removed joint l_hip_yaw
- removed joint l_knee_pitch
- removed joint l_shoulder_pitch
- removed joint l_shoulder_roll
- removed joint l_shoulder_yaw
- removed joint l_wrist_pitch
- removed joint l_wrist_roll
- removed joint l_wrist_yaw
- removed joint r_ankle_pitch
- removed joint r_ankle_roll
- removed joint r_elbow_pitch
- removed joint r_hip_pitch
- removed joint r_hip_roll
- removed joint r_hip_yaw
- removed joint r_knee_pitch
- removed joint r_shoulder_pitch
- removed joint r_shoulder_roll
- removed joint r_shoulder_yaw
- removed joint r_wrist_pitch
- removed joint r_wrist_roll
- removed joint r_wrist_yaw
- added joint joint_left_ankle_pitch: type revolute, parent link_left_shank_pitch, child link_left_foot_pitch, origin xyz=0 0 -0.339999992262544 rpy=0 0 0, axis 0 1 0, limit lower=-1.05 upper=0.52 effort=15 velocity=20.32
- added joint joint_left_ankle_roll: type revolute, parent link_left_foot_pitch, child link_left_foot_roll, origin xyz=0 0 0 rpy=0 0 0, axis 1 0 0, limit lower=-0.44 upper=0.44 effort=30 velocity=20.32
- added joint joint_left_elbow_pitch: type revolute, parent link_left_upper_arm_yaw, child link_left_lower_arm_pitch, origin xyz=0 0.00125501157055688 -0.188749174791823 rpy=0 0 0, axis 0 1 0, limit lower=-2.27 upper=2.27 effort=30 velocity=7.33
- added joint joint_left_hip_pitch: type revolute, parent link_left_thigh_yaw, child link_left_thigh_pitch, origin xyz=0 0 -0.109999999999336 rpy=0 0 0, axis 0 1 0, limit lower=-1.75 upper=0.7 effort=160 velocity=37.38
- added joint joint_left_hip_roll: type revolute, parent base, child link_left_thigh_roll, origin xyz=-0.0480000000000005 0.105 -0.0575 rpy=0 0 0, axis 1 0 0, limit lower=-0.09 upper=0.79 effort=80 velocity=12.15
- added joint joint_left_hip_yaw: type revolute, parent link_left_thigh_roll, child link_left_thigh_yaw, origin xyz=0.048 0 -0.0304999999999989 rpy=0 0 0, axis 0 0 1, limit lower=-0.7 upper=0.7 effort=60 velocity=16.76
- added joint joint_left_knee_pitch: type revolute, parent link_left_thigh_pitch, child link_left_shank_pitch, origin xyz=0 0 -0.359995124115987 rpy=0 0 0, axis 0 1 0, limit lower=-0.09 upper=1.92 effort=160 velocity=37.38
- added joint joint_left_shoulder_pitch: type revolute, parent link_torso, child link_left_upper_arm_pitch, origin xyz=0 0.126623540943386 0.0590455268445764 rpy=0.436334785573203 0 0, axis 0 1 0, limit lower=-2.79 upper=1.92 effort=38 velocity=9.11
- added joint joint_left_shoulder_roll: type revolute, parent link_left_upper_arm_pitch, child link_left_upper_arm_roll, origin xyz=0 0.0669999999997965 0 rpy=-0.436334785573203 0 0, axis 1 0 0, limit lower=-0.57 upper=3.27 effort=38 velocity=9.11
- added joint joint_left_shoulder_yaw: type revolute, parent link_left_upper_arm_roll, child link_left_upper_arm_yaw, origin xyz=0 0.040381430445538 -0.0572327709897897 rpy=0 0 0, axis 0 0 1, limit lower=-2.97 upper=2.97 effort=30 velocity=7.33
- added joint joint_left_wrist_pitch: type revolute, parent link_left_hand_roll, child link_left_hand_pitch, origin xyz=0 0 0 rpy=0 0 0, axis 0 1 0, limit lower=-0.61 upper=0.61 effort=3.95 velocity=27.96
- added joint joint_left_wrist_roll: type revolute, parent link_left_hand_yaw, child link_left_hand_roll, origin xyz=0 0.00133699944291396 -0.20107985186864 rpy=0 0 0, axis 1 0 0, limit lower=-0.96 upper=0.87 effort=3.95 velocity=27.96
- added joint joint_left_wrist_yaw: type revolute, parent link_left_lower_arm_pitch, child link_left_hand_yaw, origin xyz=0 0.000299612107771352 -0.0404989031042769 rpy=0 0 0, axis 0 0 1, limit lower=-2.97 upper=2.97 effort=10.2 velocity=24.4
- added joint joint_right_ankle_pitch: type revolute, parent link_right_shank_pitch, child link_right_foot_pitch, origin xyz=0 0 -0.339999999788054 rpy=0 0 0, axis 0 1 0, limit lower=-1.05 upper=0.52 effort=15 velocity=20.32
- added joint joint_right_ankle_roll: type revolute, parent link_right_foot_pitch, child link_right_foot_roll, origin xyz=0 0 0 rpy=0 0 0, axis 1 0 0, limit lower=-0.44 upper=0.44 effort=30 velocity=20.32
- added joint joint_right_elbow_pitch: type revolute, parent link_right_upper_arm_yaw, child link_right_lower_arm_pitch, origin xyz=0 0 -0.188530330300762 rpy=0 0 0, axis 0 1 0, limit lower=-2.27 upper=2.27 effort=30 velocity=7.33
- added joint joint_right_hip_pitch: type revolute, parent link_right_thigh_yaw, child link_right_thigh_pitch, origin xyz=0 0 -0.109999999999337 rpy=0 0 0, axis 0 1 0, limit lower=-1.75 upper=0.7 effort=160 velocity=37.38
- added joint joint_right_hip_roll: type revolute, parent base, child link_right_thigh_roll, origin xyz=-0.0480000000000003 -0.105 -0.0575 rpy=0 0 0, axis 1 0 0, limit lower=-0.79 upper=0.09 effort=80 velocity=12.15
- added joint joint_right_hip_yaw: type revolute, parent link_right_thigh_roll, child link_right_thigh_yaw, origin xyz=0.0480000000000212 0 -0.0305000000000011 rpy=0 0 0, axis 0 0 1, limit lower=-0.7 upper=0.7 effort=60 velocity=16.76
- added joint joint_right_knee_pitch: type revolute, parent link_right_thigh_pitch, child link_right_shank_pitch, origin xyz=0 0 -0.359995124115985 rpy=0 0 0, axis 0 1 0, limit lower=-0.09 upper=1.92 effort=160 velocity=37.38
- added joint joint_right_shoulder_pitch: type revolute, parent link_torso, child link_right_upper_arm_pitch, origin xyz=0 -0.126623540926852 0.0590455268368039 rpy=-0.436332306093773 0 0, axis 0 1 0, limit lower=-2.79 upper=1.92 effort=38 velocity=9.11
- added joint joint_right_shoulder_roll: type revolute, parent link_right_upper_arm_pitch, child link_right_upper_arm_roll, origin xyz=0 -0.0670000000000026 0 rpy=0.436332306093773 0 0, axis 1 0 0, limit lower=-3.27 upper=0.57 effort=38 velocity=9.11
- added joint joint_right_shoulder_yaw: type revolute, parent link_right_upper_arm_roll, child link_right_upper_arm_yaw, origin xyz=0 -0.039999999998954 -0.0575000000000302 rpy=0 0 0, axis 0 0 1, limit lower=-2.97 upper=2.97 effort=30 velocity=7.33
- added joint joint_right_wrist_pitch: type revolute, parent link_right_hand_roll, child link_right_hand_pitch, origin xyz=0 0 0 rpy=0 0 0, axis 0 1 0, limit lower=-0.61 upper=0.61 effort=3.95 velocity=27.96
- added joint joint_right_wrist_roll: type revolute, parent link_right_hand_yaw, child link_right_hand_roll, origin xyz=0 0 -0.201084296746609 rpy=0 0 0, axis 1 0 0, limit lower=-0.87 upper=0.96 effort=3.95 velocity=27.96
- added joint joint_right_wrist_yaw: type revolute, parent link_right_lower_arm_pitch, child link_right_hand_yaw, origin xyz=0 -3.03303104252084E-05 -0.0404999999922469 rpy=0 0 0, axis 0 0 1, limit lower=-2.97 upper=2.97 effort=10.2 velocity=24.4

Commit message: update gr1t2 mjcf

File: models/GR1/GR1T2/urdf/GR1T2_raw.urdf (robot description, URDF)
Before this commit: robot GR1T2, 35 links, 34 joints
Links:
- removed link l_shank_pitch
- removed link l_thigh_roll
- added link link_left_shank_pitch, mass 2.4196; collision mesh filename=../meshes/l_shank_pitch.STL; visual mesh filename=../meshes/l_shank_pitch.STL
- added link link_left_thigh_roll, mass 1.24083588; collision mesh filename=../meshes/l_thigh_roll.STL; visual mesh filename=../meshes/l_thigh_roll.STL

Commit message: fix bugs

File: models/GR1/GR1T2/urdf/GR1T2_raw.urdf (robot description, URDF)
Before this commit: robot GR1T2, 35 links, 34 joints
Links:
- link link_waist_pitch: geometry collision mesh filename=../meshes/waist_pitch.STL; visual mesh filename=../meshes/waist_pitch.STL
